File: hardware/pcbDesign/ph-sensor.kicad_sch (KiCad schematic)
At the start: 21 parts, among them J1 DURAFET_INPUT, SW1 SW_Reed, U1 ADS1115, U1 DS3231, U2 ADS1015, U2 NRF24L01

Commit message: V1 JLCPCB design
Parts:
- removed BT1, BT2: 3.6V, symbol Device:Battery_Cell
- added C5: C, Capacitor_SMD:C_1206_3216Metric_Pad1.33x1.80mm_HandSolder, symbol Device:C
- added J2: Conn_01x03_Pin, Connector_PinSocket_2.54mm:PinSocket_1x03_P2.54mm_Horizontal, symbol Connector:Conn_01x03_Pin
- A1: footprint Module:Adafruit_Feather -> Library:Adalogger_amelia_nomount
- C1: value 20uF -> C; footprint (none) -> Capacitor_SMD:C_1206_3216Metric_Pad1.33x1.80mm_HandSolder
- C2, C3, C4: value 100uF -> C; footprint (none) -> Capacitor_SMD:C_1206_3216Metric_Pad1.33x1.80mm_HandSolder
- J1: value DURAFET_INPUT -> Conn_01x06_Pin; footprint (none) -> Connector_PinSocket_2.54mm:PinSocket_1x06_P2.54mm_Horizontal
- R1, R4, R5, R6, R7: value 1M -> R_US; footprint (none) -> Resistor_SMD:R_0603_1608Metric_Pad0.98x0.95mm_HandSolder
- R2, R3: value 10k -> R_US; footprint (none) -> Resistor_SMD:R_0603_1608Metric_Pad0.98x0.95mm_HandSolder
- R8: value 15k -> R_US; footprint (none) -> Resistor_SMD:R_0603_1608Metric_Pad0.98x0.95mm_HandSolder
- SW1: footprint (none) -> Library:REED_amelia
- U1: value DS3231 -> DS3231MZ; footprint Package_SO:SOIC-8_3.9x4.9mm_P1.27mm -> Library:DS3231RTC_amelia
- U1: value ADS1115 -> ADS_Ritger; footprint Package_SO:TSSOP-10_3x3mm_P0.5mm -> Library:ADC_amelia_nomount; symbol Analog_ADC:ADS1115IDGS -> Analog_ADC:ADS_Ritger
- U2: value ADS1015 -> ADS_Ritger; footprint Package_SO:TSSOP-10_3x3mm_P0.5mm -> Library:ADC_amelia_nomount; symbol Analog_ADC:ADS1015IDGS -> Analog_ADC:ADS_Ritger
- U2: value NRF24L01 -> NRF24L01_Breakout; footprint RF_Module:nRF24L01_Breakout -> Library:NRF24L01Module
Connections:
- net GND: now also U1.10 (AIN1), U1.2 (GND), U1.6 (GND), U2.10 (AIN1), U2.2 (GND), C5.2, J2.3 (Pin_3); no longer C2.1, J1.5 (Pin_5), R6.2, U1.3 (GND), U1.5 (AIN1), U1.5 (GND), U1.6 (AIN2), U2.1 (ADDR), U2.3 (GND)
- net MISO: now also A1.13 (MISO/D22)
- net MOSI: no longer A1.13 (MISO/D22)
- net SCL: now also U1.3 (SCL), U1.3 (SCL), U2.3 (SCL); no longer U1.10 (SCL), U1.8 (SCL), U2.10 (SCL)
- net SDA: now also U1.4 (SDA), U1.4 (SDA), U2.4 (SDA); no longer U1.7 (SDA), U1.9 (SDA), U2.9 (SDA)
- net pH: now also J1.4 (Pin_4), U1.11 (AIN0); no longer J1.1 (Pin_1), U1.4 (AIN0)
- net at A1.19 (D5): now also U1.2 (~{INT}/SQW); no longer U1.3 (~{INT}/SQW)
- net at R7.1, R8.2: now also U1.8 (AIN3); no longer U1.7 (AIN3)
- net at C4.1, R1.2, R2.1: now also U2.11 (AIN0); no longer U2.4 (AIN0)
- net at C3.1, R3.1, R4.2: now also U2.9 (AIN2); no longer U2.6 (AIN2)
- net +3V3 renamed +BATT
- net +BATT: now also J1.1 (Pin_1), U1.5 (ADDR), U1.5 (VCC), U2.1 (VDD), C5.1, J2.1 (Pin_1); no longer J1.2 (Pin_2), U1.2 (VCC), U1.8 (VDD), U2.8 (VDD)
- net Batt- renamed -BATT
- net -BATT: now also J1.2 (Pin_2), J2.2 (Pin_2); no longer J1.4 (Pin_4)
- new net RTH_High: C2.1, J1.5 (Pin_5), R6.2, U1.9 (AIN2)
- no-connect marks 23 -> 25
Other:
- moved on the sheet: C1, C2, C4, R2, R5, R6, R7, R8
