File: hardware/test/ph-sensor_newschem.kicad_sch (KiCad schematic)
At the start: 21 parts, among them J1 Conn_01x06_Pin, J2 Conn_01x03_Pin, SW1 SW_Reed, U1 ADS_Ritger, U1 DS3231MZ, U2 ADS_Ritger, U2 NRF24L01_Breakout

Commit message: update pcb schematic/design
Parts:
- C1: value 22uF -> C
- C2, C3, C4: value 100uF -> C
- C5: value 10uF -> C
- R1, R4, R5, R6, R7: value 1M -> R_US
- R2, R3: value 10k -> R_US
- R8: value 15k -> R_US
Connections:
- net +BATT: now also U1.5 (VCC), U2.2 (VCC); no longer U1.2 (VCC), U2.1 (VCC)
- net GND: now also U1.6 (GND), U2.1 (GND); no longer U1.1 (GND), U1.8 (AIN3), U2.9 (GND)
- net MISO: now also U2.7 (MISO); no longer U2.8 (MISO)
- net MOSI: now also U2.6 (MOSI); no longer U2.5 (MOSI)
- net SCK: now also U2.5 (SCK); no longer U2.6 (SCK)
- net SCL: now also U1.3 (SCL); no longer U1.4 (SCL)
- net SDA: now also U1.4 (SDA); no longer U1.3 (SDA)
- net at A1.19 (D5): now also U1.2 (~{INT}/SQW); no longer U1.5 (~{INT}/SQW)
- net at R7.1, R8.2: now also U1.8 (AIN3)
- net at A1.20 (D6): now also U2.3 (CE); no longer U2.4 (CE)
- net at A1.22 (D10): now also U2.4 (~{CSN}); no longer U2.3 (~{CSN})
- no-connect marks 27 -> 25
